File: KiCAD Project/5V Regulator.kicad_sch (KiCad schematic)
At the start: 20 parts, among them U1 LM64440APPQRYFRQ1

Commit message: v1.0.0 RC3
Minor change to upstream USB port to connect Vbus to ESD protection vice on-board 5V.
Parts:
- C12: value GRM0225C1C100FA03L -> VJ0402A100GXJCW1BC; Height 0.25 -> 0.5; Manufacturer_Name Murata -> Vishay; Manufacturer_Part_Number GRM0225C1C100FA03L -> VJ0402A100GXJCW1BC; Mouser Part Number 81-GRM0225C1C100FA03 -> 77-VJ0402A100GXJCBC; Mouser Price/Stock https://www.mouser.com/ProductDetail/Murata-Electronics/GRM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 -> https://www.mouser.com/ProductDetail/77-VJ0402A100GXJCBC
Changed lines of the file:
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@@
 		(title "1026 RPi Power Hat")
 		(date "2025-04-11")
-		(rev "1")
+		(rev "1.0.0 RC3")
 		(company "Dan Wilson")
 		(comment 1 "Copyright © 2025 Dan Wilson")
@@
 			)
 		)
-		(property "Value" "GRM0225C1C100FA03L"
+		(property "Value" "VJ0402A100GXJCW1BC"
 			(at 192.659 99.1179 0)
 			(effects
@@
 			)
 		)
-		(property "Datasheet" "https://www.mouser.com/datasheet/2/281/GRM0225C1C100FA03_01A-1978859.pdf"
+		(property "Datasheet" "https://www.vishay.com/doc?28548"
 			(at 195.58 100.33 0)
 			(effects
@@
 			)
 		)
-		(property "Height" "0.25"
+		(property "Height" "0.5"
 			(at 195.58 100.33 0)
 			(effects
@@
 			)
 		)
-		(property "Manufacturer_Name" "Murata"
+		(property "Manufacturer_Name" "Vishay"
 			(at 195.58 100.33 0)
 			(effects
@@
 			)
 		)
-		(property "Manufacturer_Part_Number" "GRM0225C1C100FA03L"
+		(property "Manufacturer_Part_Number" "VJ0402A100GXJCW1BC"
 			(at 195.58 100.33 0)
 			(effects
@@
 			)
 		)
-		(property "Mouser Part Number" "81-GRM0225C1C100FA03"
+		(property "Mouser Part Number" "77-VJ0402A100GXJCBC"
 			(at 195.58 100.33 0)
 			(effects
@@
 			)
 		)
-		(property "Mouser Price/Stock" "https://www.mouser.com/ProductDetail/Murata-Electronics/GRM0225C1C100FA03L?qs=rrS6PyfT74dMR%2FKublCCEA%3D%3D"
+		(property "Mouser Price/Stock" "https://www.mouser.com/ProductDetail/77-VJ0402A100GXJCBC"
 			(at 195.58 100.33 0)
 			(effects

Commit message: v1.0.0A
Moved all symbols, footprints, and 3D models to local project-specific libraries in /KiCAD Project/Libraries.
Parts:
- C10, C11, C3, C4: footprint Capacitor_SMD:C_1210_3225Metric -> 1026-3D:C_1210_3225Metric; symbol Device:C -> 1026-3D:C
- C12, C5, C6, C8, C9: footprint Capacitor_SMD:C_0402_1005Metric -> 1026-3D:C_0402_1005Metric; symbol Device:C -> 1026-3D:C
- C7: footprint Capacitor_SMD:C_0603_1608Metric -> 1026-3D:C_0603_1608Metric; symbol Device:C -> 1026-3D:C
- D4: footprint DW_Optoelectronics:[D] Wurth Elektronik 150040RS73240 -> 1026-3D:[D] Wurth Elektronik 150040RS73240; symbol DW_Optoelectronics:[D] Wurth Elektronik 150040RS73240 -> 1026-3D:[D] Wurth Elektronik 150040RS73240
- L2: footprint DW_Passives:[L] Coilcraft Inductor XGL4025 -> 1026-3D:[L] Coilcraft Inductor XGL4025; symbol DW_Passives:[L] Coilcraft Inductor XGL4025 1.5uH 11mohm -> 1026-3D:[L] Coilcraft Inductor XGL4025 1.5uH 11mohm
- R3, R4, R5, R6, R7, R8, R9: footprint Resistor_SMD:R_0402_1005Metric -> 1026-3D:R_0402_1005Metric; symbol Device:R_US -> 1026-3D:R_US
- U1: footprint DW_Semiconductors:[U] TI LM63460 Sw Volt Reg -> 1026-3D:[U] TI LM63460 Sw Volt Reg; symbol DW_Semiconductors:[U] TI LM64440 Sw Volt Reg -> 1026-3D:[U] TI LM64440 Sw Volt Reg
Changed lines of the file:
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@@
 	)
 	(symbol
-		(lib_id "Device:C")
+		(lib_id "1026-3D:C")
 		(at 162.56 97.79 180)
 		(unit 1)
@@
 			)
 		)
-		(property "Footprint" "Capacitor_SMD:C_0402_1005Metric"
+		(property "Footprint" "1026-3D:C_0402_1005Metric"
 			(at 161.5948 93.98 0)
 			(effects
@@
 	)
 	(symbol
-		(lib_id "Device:C")
+		(lib_id "1026-3D:C")
 		(at 215.9 87.63 0)
 		(unit 1)
@@
 			)
 		)
-		(property "Footprint" "Capacitor_SMD:C_1210_3225Metric"
+		(property "Footprint" "1026-3D:C_1210_3225Metric"
 			(at 216.8652 91.44 0)
 			(effects
@@
 	)
 	(symbol
-		(lib_id "Device:R_US")
+		(lib_id "1026-3D:R_US")
 		(at 195.58 87.63 0)
 		(unit 1)
@@
 			)
 		)
-		(property "Footprint" "Resistor_SMD:R_0402_1005Metric"
+		(property "Footprint" "1026-3D:R_0402_1005Metric"
 			(at 196.596 87.884 90)
 			(effects
@@
 	)
 	(symbol
-		(lib_id "Device:R_US")
+		(lib_id "1026-3D:R_US")
 		(at 118.11 50.8 90)
 		(unit 1)
@@
 			)
 		)
-		(property "Footprint" "Resistor_SMD:R_0402_1005Metric"
+		(property "Footprint" "1026-3D:R_0402_1005Metric"
 			(at 118.364 49.784 90)
 			(effects
@@
 	)
 	(symbol
-		(lib_id "Device:C")
+		(lib_id "1026-3D:C")
 		(at 71.12 72.39 0)
 		(unit 1)
@@
 			)
 		)
-		(property "Footprint" "Capacitor_SMD:C_1210_3225Metric"
+		(property "Footprint" "1026-3D:C_1210_3225Metric"
 			(at 72.0852 76.2 0)
 			(effects
@@
 	)
 	(symbol
-		(lib_id "power:GND")
+		(lib_id "1026-3D:GND")
 		(at 76.2 127 0)
 		(unit 1)
@@
 	)
 	(symbol
-		(lib_id "DW_Optoelectronics:[D] Wurth Elektronik 150040RS73240")
+		(lib_id "1026-3D:[D] Wurth Elektronik 150040RS73240")
 		(at 152.4 50.8 180)
 		(unit 1)
@@
 			)
 		)
-		(property "Footprint" "DW_Optoelectronics:[D] Wurth Elektronik 150040RS73240"
+		(property "Footprint" "1026-3D:[D] Wurth Elektronik 150040RS73240"
 			(at 139.7 -42.85 0)
 			(effects
@@
 	)
 	(symbol
-		(lib_id "Device:C")
+		(lib_id "1026-3D:C")
 		(at 228.6 87.63 0)
 		(unit 1)
@@
 			)
 		)
-		(property "Footprint" "Capacitor_SMD:C_1210_3225Metric"
+		(property "Footprint" "1026-3D:C_1210_3225Metric"
 			(at 229.5652 91.44 0)
 			(effects
@@
 	)
 	(symbol
-		(lib_id "Device:C")
+		(lib_id "1026-3D:C")
 		(at 86.36 72.39 0)
 		(unit 1)
@@
 			)
 		)
-		(property "Footprint" "Capacitor_SMD:C_0402_1005Metric"
+		(property "Footprint" "1026-3D:C_0402_1005Metric"
 			(at 87.3252 76.2 0)
 			(effects
@@
 	)
 	(symbol
-		(lib_id "Device:C")
+		(lib_id "1026-3D:C")
 		(at 175.26 88.9 90)
 		(unit 1)
@@
 			)
 		)
-		(property "Footprint" "Capacitor_SMD:C_0402_1005Metric"
+		(property "Footprint" "1026-3D:C_0402_1005Metric"
 			(at 179.07 87.9348 0)
 			(effects
@@
 	)
 	(symbol
-		(lib_id "Device:C")
+		(lib_id "1026-3D:C")
 		(at 93.98 72.39 0)
 		(unit 1)
@@
 			)
 		)
-		(property "Footprint" "Capacitor_SMD:C_0402_1005Metric"
+		(property "Footprint" "1026-3D:C_0402_1005Metric"
 			(at 94.9452 76.2 0)
 			(effects
@@
 	)
 	(symbol
-		(lib_id "Device:C")
+		(lib_id "1026-3D:C")
 		(at 76.2 105.41 0)
 		(unit 1)
@@
 			)
 		)
-		(property "Footprint" "Capacitor_SMD:C_0603_1608Metric"
+		(property "Footprint" "1026-3D:C_0603_1608Metric"
 			(at 77.1652 109.22 0)
 			(effects
@@
 	)
 	(symbol
-		(lib_id "Device:R_US")
+		(lib_id "1026-3D:R_US")
 		(at 203.2 92.71 0)
 		(unit 1)
@@
 			)
 		)
-		(property "Footprint" "Resistor_SMD:R_0402_1005Metric"
+		(property "Footprint" "1026-3D:R_0402_1005Metric"
 			(at 204.216 92.964 90)
 			(effects
@@
 	)
 	(symbol
-		(lib_id "Device:R_US")
+		(lib_id "1026-3D:R_US")
 		(at 203.2 115.57 180)
 		(unit 1)
@@
 			)
 		)
-		(property "Footprint" "Resistor_SMD:R_0402_1005Metric"
+		(property "Footprint" "1026-3D:R_0402_1005Metric"
 			(at 202.184 115.316 90)
 			(effects
@@
 	)
 	(symbol
-		(lib_id "Device:R_US")
+		(lib_id "1026-3D:R_US")
 		(at 63.5 95.25 0)
 		(unit 1)
@@
 			)
 		)
-		(property "Footprint" "Resistor_SMD:R_0402_1005Metric"
+		(property "Footprint" "1026-3D:R_0402_1005Metric"
 			(at 64.516 95.504 90)
 			(effects
@@
 	)
 	(symbol
-		(lib_id "Device:R_US")
+		(lib_id "1026-3D:R_US")
 		(at 63.5 82.55 0)
 		(unit 1)
@@
 			)
 		)
-		(property "Footprint" "Resistor_SMD:R_0402_1005Metric"
+		(property "Footprint" "1026-3D:R_0402_1005Metric"
 			(at 64.516 82.804 90)
 			(effects
@@
 	)
 	(symbol
-		(lib_id "Device:C")
+		(lib_id "1026-3D:C")
 		(at 78.74 72.39 0)
 		(unit 1)
@@
 			)
 		)
-		(property "Footprint" "Capacitor_SMD:C_1210_3225Metric"
+		(property "Footprint" "1026-3D:C_1210_3225Metric"
 			(at 79.7052 76.2 0)
 			(effects
@@
 	)
 	(symbol
-		(lib_id "Device:C")
+		(lib_id "1026-3D:C")
 		(at 195.58 100.33 180)
 		(unit 1)
@@
 			)
 		)
-		(property "Footprint" "Capacitor_SMD:C_0402_1005Metric"
+		(property "Footprint" "1026-3D:C_0402_1005Metric"
 			(at 194.6148 96.52 0)
 			(effects
@@
 	)
 	(symbol
-		(lib_id "Device:R_US")
+		(lib_id "1026-3D:R_US")
 		(at 175.26 67.31 90)
 		(unit 1)
@@
 			)
 		)
-		(property "Footprint" "Resistor_SMD:R_0402_1005Metric"
+		(property "Footprint" "1026-3D:R_0402_1005Metric"
 			(at 175.514 66.294 90)
 			(effects
@@
 	)
 	(symbol
-		(lib_id "DW_Passives:[L] Coilcraft Inductor XGL4025 1.5uH 11mohm")
+		(lib_id "1026-3D:[L] Coilcraft Inductor XGL4025 1.5uH 11mohm")
 		(at 165.1 78.74 0)
 		(unit 1)
@@
 			)
 		)
-		(property "Footprint" "DW_Passives:[L] Coilcraft Inductor XGL4025"
+		(property "Footprint" "1026-3D:[L] Coilcraft Inductor XGL4025"
 			(at 181.61 174.93 0)
 			(effects
@@
 	)
 	(symbol
-		(lib_id "DW_Semiconductors:[U] TI LM64440 Sw Volt Reg")
+		(lib_id "1026-3D:[U] TI LM64440 Sw Volt Reg")
 		(at 101.6 66.04 0)
 		(unit 1)
@@
 			)
 		)
-		(property "Footprint" "DW_Semiconductors:[U] TI LM63460 Sw Volt Reg"
+		(property "Footprint" "1026-3D:[U] TI LM63460 Sw Volt Reg"
 			(at 127 127 0)
 			(effects
