File: KiCAD Project/Linear Regulators.kicad_sch (KiCad schematic)
At the start: 10 parts, among them U2 TLV75511PDQNR, U3 TLV75533PDQNR

Commit message: v1.0.0 RC2
Build candidate 2
Parts:
- R10, R11: Height 0.40 -> 0.35
Changed lines of the file:
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@@
 			)
 		)
-		(property "Datasheet" "https://www.vishay.com/doc?20035"
+		(property "Datasheet" "https://www.vishay.com/docs/28773/crcwce3.pdf"
 			(at 82.55 87.63 0)
 			(effects
@@
 			)
 		)
-		(property "Height" "0.40"
+		(property "Height" "0.35"
 			(at 82.55 87.63 0)
 			(effects
@@
 			)
 		)
-		(property "Datasheet" "https://www.vishay.com/doc?20035"
+		(property "Datasheet" "https://www.vishay.com/docs/28773/crcwce3.pdf"
 			(at 82.55 71.12 0)
 			(effects
@@
 			)
 		)
-		(property "Height" "0.40"
+		(property "Height" "0.35"
 			(at 82.55 71.12 0)
 			(effects

Commit message: v1.0.0A
Moved all symbols, footprints, and 3D models to local project-specific libraries in /KiCAD Project/Libraries.
Parts:
- C13, C14, C15, C16: footprint Capacitor_SMD:C_0603_1608Metric -> 1026-3D:C_0603_1608Metric; symbol Device:C -> 1026-3D:C
- R10, R11, R12, R13: footprint Resistor_SMD:R_0402_1005Metric -> 1026-3D:R_0402_1005Metric; symbol Device:R_US -> 1026-3D:R_US
- U2: footprint DW_Semiconductors:[U] TI LDO Regulator TLV755 DQN -> 1026-3D:[U] TI LDO Regulator TLV755 DQN; symbol DW_Semiconductors:[U] TI LDO Regulator TLV75511PDQNR -> 1026-3D:[U] TI LDO Regulator TLV75511PDQNR
- U3: footprint DW_Semiconductors:[U] TI LDO Regulator TLV755 DQN -> 1026-3D:[U] TI LDO Regulator TLV755 DQN; symbol DW_Semiconductors:[U] TI LDO Regulator TLV75533PDQNR -> 1026-3D:[U] TI LDO Regulator TLV75533PDQNR
Changed lines of the file:
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@@
 	)
 	(symbol
-		(lib_id "Device:C")
+		(lib_id "1026-3D:C")
 		(at 165.1 69.85 0)
 		(unit 1)
@@
 			)
 		)
-		(property "Footprint" "Capacitor_SMD:C_0603_1608Metric"
+		(property "Footprint" "1026-3D:C_0603_1608Metric"
 			(at 166.0652 73.66 0)
 			(effects
@@
 	)
 	(symbol
-		(lib_id "DW_Semiconductors:[U] TI LDO Regulator TLV75533PDQNR")
+		(lib_id "1026-3D:[U] TI LDO Regulator TLV75533PDQNR")
 		(at 132.08 118.11 0)
 		(unit 1)
@@
 			)
 		)
-		(property "Footprint" "DW_Semiconductors:[U] TI LDO Regulator TLV755 DQN"
+		(property "Footprint" "1026-3D:[U] TI LDO Regulator TLV755 DQN"
 			(at 132.08 139.7 0)
 			(effects
@@
 	)
 	(symbol
-		(lib_id "Device:C")
+		(lib_id "1026-3D:C")
 		(at 101.6 69.85 0)
 		(unit 1)
@@
 			)
 		)
-		(property "Footprint" "Capacitor_SMD:C_0603_1608Metric"
+		(property "Footprint" "1026-3D:C_0603_1608Metric"
 			(at 102.5652 73.66 0)
 			(effects
@@
 	)
 	(symbol
-		(lib_id "Device:R_US")
+		(lib_id "1026-3D:R_US")
 		(at 82.55 87.63 0)
 		(unit 1)
@@
 			)
 		)
-		(property "Footprint" "Resistor_SMD:R_0402_1005Metric"
+		(property "Footprint" "1026-3D:R_0402_1005Metric"
 			(at 83.566 87.884 90)
 			(effects
@@
 	)
 	(symbol
-		(lib_id "Device:R_US")
+		(lib_id "1026-3D:R_US")
 		(at 82.55 138.43 0)
 		(unit 1)
@@
 			)
 		)
-		(property "Footprint" "Resistor_SMD:R_0402_1005Metric"
+		(property "Footprint" "1026-3D:R_0402_1005Metric"
 			(at 83.566 138.684 90)
 			(effects
@@
 	)
 	(symbol
-		(lib_id "power:GND")
+		(lib_id "1026-3D:GND")
 		(at 101.6 88.9 0)
 		(unit 1)
@@
 	)
 	(symbol
-		(lib_id "Device:R_US")
+		(lib_id "1026-3D:R_US")
 		(at 82.55 71.12 0)
 		(unit 1)
@@
 			)
 		)
-		(property "Footprint" "Resistor_SMD:R_0402_1005Metric"
+		(property "Footprint" "1026-3D:R_0402_1005Metric"
 			(at 83.566 71.374 90)
 			(effects
@@
 	)
 	(symbol
-		(lib_id "Device:C")
+		(lib_id "1026-3D:C")
 		(at 165.1 120.65 0)
 		(unit 1)
@@
 			)
 		)
-		(property "Footprint" "Capacitor_SMD:C_0603_1608Metric"
+		(property "Footprint" "1026-3D:C_0603_1608Metric"
 			(at 166.0652 124.46 0)
 			(effects
@@
 	)
 	(symbol
-		(lib_id "DW_Semiconductors:[U] TI LDO Regulator TLV75511PDQNR")
+		(lib_id "1026-3D:[U] TI LDO Regulator TLV75511PDQNR")
 		(at 132.08 67.31 0)
 		(unit 1)
@@
 			)
 		)
-		(property "Footprint" "DW_Semiconductors:[U] TI LDO Regulator TLV755 DQN"
+		(property "Footprint" "1026-3D:[U] TI LDO Regulator TLV755 DQN"
 			(at 132.08 88.9 0)
 			(effects
@@
 	)
 	(symbol
-		(lib_id "Device:C")
+		(lib_id "1026-3D:C")
 		(at 101.6 120.65 0)
 		(unit 1)
@@
 			)
 		)
-		(property "Footprint" "Capacitor_SMD:C_0603_1608Metric"
+		(property "Footprint" "1026-3D:C_0603_1608Metric"
 			(at 102.5652 124.46 0)
 			(effects
@@
 	)
 	(symbol
-		(lib_id "Device:R_US")
+		(lib_id "1026-3D:R_US")
 		(at 82.55 121.92 0)
 		(unit 1)
@@
 			)
 		)
-		(property "Footprint" "Resistor_SMD:R_0402_1005Metric"
+		(property "Footprint" "1026-3D:R_0402_1005Metric"
 			(at 83.566 122.174 90)
 			(effects
@@
 	)
 	(symbol
-		(lib_id "power:GND")
+		(lib_id "1026-3D:GND")
 		(at 101.6 139.7 0)
 		(unit 1)
