File: KiCAD Project/Mechanical.kicad_sch (KiCad schematic)
At the start: 10 parts, among them P1 DW_PCB_Logo, P2 Raspberry Pi HAT+ Designator

Commit message: v1.0.0 RC2
Build candidate 2
Parts:
- G1, P1, P2: now left out of the parts list
Changed lines of the file:
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@@
 		(unit 1)
 		(exclude_from_sim no)
-		(in_bom yes)
+		(in_bom no)
 		(on_board yes)
 		(dnp no)
@@
 		(unit 1)
 		(exclude_from_sim no)
-		(in_bom yes)
+		(in_bom no)
 		(on_board yes)
 		(dnp no)
@@
 		(unit 1)
 		(exclude_from_sim no)
-		(in_bom yes)
-		(on_board yes)
-		(dnp no)
+		(in_bom no)
+		(on_board yes)
+		(dnp no)

Commit message: v1.0.0
Initial Commit
Parts:
- added G2: OSHW_Logo, DW_Mechanical:OSHW_Logo, symbol DW_Mechanical:OSHW_Logo
- H1, H4: footprint DW_Mechanical:[MH] MountingHole_2.7mm_M2.5_Pad_StencilRegHole -> DW_Mechanical:[MH] MountingHole_2.7mm_M2.5
- H2, H3: footprint DW_Mechanical:[MH] MountingHole_2.7mm_M2.5_Pad -> DW_Mechanical:[MH] MountingHole_2.7mm_M2.5_StencilRegHole
Changed lines of the file:
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@@
 	(title_block
 		(title "1026 RPi Power Hat")
-		(date "2025-04-11")
-		(rev "1.0.0 RC3")
+		(date "2025-05-18")
+		(rev "1.0.0")
 		(company "Dan Wilson")
 		(comment 1 "Copyright © 2025 Dan Wilson")
@@
 	(symbol
 		(lib_id "Mechanical:MountingHole")
-		(at 106.68 96.52 0)
-		(unit 1)
-		(exclude_from_sim no)
-		(in_bom no)
-		(on_board yes)
-		(dnp no)
-		(fields_autoplaced yes)
-		(property "Reference" "H2"
-			(at 109.22 95.3078 0)
+		(at 101.6 88.9 0)
+		(unit 1)
+		(exclude_from_sim no)
+		(in_bom no)
+		(on_board yes)
+		(dnp no)
+		(fields_autoplaced yes)
+		(property "Reference" "H1"
+			(at 104.14 87.6878 0)
 			(effects
 				(font
@@
 		)
 		(property "Value" "MountingHole"
-			(at 109.22 97.7321 0)
-			(effects
-				(font
-					(size 1.27 1.27)
-				)
-				(justify left)
-			)
-		)
-		(property "Footprint" "DW_Mechanical:[MH] MountingHole_2.7mm_M2.5_Pad"
-			(at 106.68 96.52 0)
+			(at 104.14 90.1121 0)
+			(effects
+				(font
+					(size 1.27 1.27)
+				)
+				(justify left)
+			)
+		)
+		(property "Footprint" "DW_Mechanical:[MH] MountingHole_2.7mm_M2.5"
+			(at 101.6 88.9 0)
 			(effects
 				(font
@@
 		)
 		(property "Datasheet" "~"
-			(at 106.68 96.52 0)
+			(at 101.6 88.9 0)
 			(effects
 				(font
@@
 		)
 		(property "Description" "Mounting Hole without connection"
-			(at 106.68 96.52 0)
-			(effects
-				(font
-					(size 1.27 1.27)
-				)
-				(hide yes)
-			)
-		)
-		(instances
-			(project "1026 RPi Power Hat"
-				(path "/0e50632e-8a8b-4b7f-ac56-99c7667bb88a/11547498-585a-4b65-8383-0a98326c007f"
-					(reference "H2")
-					(unit 1)
-				)
-			)
-		)
-	)
-	(symbol
-		(lib_id "Mechanical:MountingHole")
-		(at 106.68 91.44 0)
-		(unit 1)
-		(exclude_from_sim no)
-		(in_bom no)
-		(on_board yes)
-		(dnp no)
-		(fields_autoplaced yes)
-		(property "Reference" "H1"
-			(at 109.22 90.2278 0)
-			(effects
-				(font
-					(size 1.27 1.27)
-				)
-				(justify left)
-			)
-		)
-		(property "Value" "MountingHole"
-			(at 109.22 92.6521 0)
-			(effects
-				(font
-					(size 1.27 1.27)
-				)
-				(justify left)
-			)
-		)
-		(property "Footprint" "DW_Mechanical:[MH] MountingHole_2.7mm_M2.5_Pad_StencilRegHole"
-			(at 106.68 91.44 0)
-			(effects
-				(font
-					(size 1.27 1.27)
-				)
-				(hide yes)
-			)
-		)
-		(property "Datasheet" "~"
-			(at 106.68 91.44 0)
-			(effects
-				(font
-					(size 1.27 1.27)
-				)
-				(hide yes)
-			)
-		)
-		(property "Description" "Mounting Hole without connection"
-			(at 106.68 91.44 0)
+			(at 101.6 88.9 0)
 			(effects
 				(font
@@
 	)
 	(symbol
-		(lib_id "Mechanical:MountingHole")
-		(at 106.68 101.6 0)
-		(unit 1)
-		(exclude_from_sim no)
-		(in_bom no)
-		(on_board yes)
-		(dnp no)
-		(fields_autoplaced yes)
-		(property "Reference" "H3"
-			(at 109.22 100.3878 0)
-			(effects
-				(font
-					(size 1.27 1.27)
-				)
-				(justify left)
-			)
-		)
-		(property "Value" "MountingHole"
-			(at 109.22 102.8121 0)
-			(effects
-				(font
-					(size 1.27 1.27)
-				)
-				(justify left)
-			)
-		)
-		(property "Footprint" "DW_Mechanical:[MH] MountingHole_2.7mm_M2.5_Pad"
-			(at 106.68 101.6 0)
-			(effects
-				(font
-					(size 1.27 1.27)
-				)
-				(hide yes)
-			)
-		)
-		(property "Datasheet" "~"
-			(at 106.68 101.6 0)
-			(effects
-				(font
-					(size 1.27 1.27)
-				)
-				(hide yes)
-			)
-		)
-		(property "Description" "Mounting Hole without connection"
-			(at 106.68 101.6 0)
+		(lib_id "DW_Mechanical:OSHW_Logo")
+		(at 165.1 101.6 0)
+		(unit 1)
+		(exclude_from_sim no)
+		(in_bom no)
+		(on_board yes)
+		(dnp no)
+		(fields_autoplaced yes)
+		(property "Reference" "G2"
+			(at 165.1 96.52 0)
+			(effects
+				(font
+					(size 1.27 1.27)
+				)
+				(hide yes)
+			)
+		)
+		(property "Value" "OSHW_Logo"
+			(at 165.1 106.68 0)
+			(effects
+				(font
+					(size 1.27 1.27)
+				)
+				(hide yes)
+			)
+		)
+		(property "Footprint" "DW_Mechanical:OSHW_Logo"
+			(at 165.1 101.6 0)
+			(effects
+				(font
+					(size 1.27 1.27)
+				)
+				(hide yes)
+			)
+		)
+		(property "Datasheet" ""
+			(at 165.1 101.6 0)
+			(effects
+				(font
+					(size 1.27 1.27)
+				)
+				(hide yes)
+			)
+		)
+		(property "Description" "Open Source Hardware Logo 8 mm"
+			(at 165.1 101.6 0)
 			(effects
 				(font
@@
 			(project "1026 RPi Power Hat"
 				(path "/0e50632e-8a8b-4b7f-ac56-99c7667bb88a/11547498-585a-4b65-8383-0a98326c007f"
-					(reference "H3")
+					(reference "G2")
 					(unit 1)
 				)
@@
 	(symbol
 		(lib_id "Mechanical:MountingHole")
-		(at 106.68 106.68 0)
-		(unit 1)
-		(exclude_from_sim no)
-		(in_bom no)
-		(on_board yes)
-		(dnp no)
-		(fields_autoplaced yes)
-		(property "Reference" "H4"
-			(at 109.22 105.4678 0)
+		(at 101.6 95.25 0)
+		(unit 1)
+		(exclude_from_sim no)
+		(in_bom no)
+		(on_board yes)
+		(dnp no)
+		(fields_autoplaced yes)
+		(property "Reference" "H2"
+			(at 104.14 94.0378 0)
 			(effects
 				(font
@@
 		)
 		(property "Value" "MountingHole"
-			(at 109.22 107.8921 0)
-			(effects
-				(font
-					(size 1.27 1.27)
-				)
-				(justify left)
-			)
-		)
-		(property "Footprint" "DW_Mechanical:[MH] MountingHole_2.7mm_M2.5_Pad_StencilRegHole"
-			(at 106.68 106.68 0)
+			(at 104.14 96.4621 0)
+			(effects
+				(font
+					(size 1.27 1.27)
+				)
+				(justify left)
+			)
+		)
+		(property "Footprint" "DW_Mechanical:[MH] MountingHole_2.7mm_M2.5_StencilRegHole"
+			(at 101.6 95.25 0)
 			(effects
 				(font
@@
 		)
 		(property "Datasheet" "~"
-			(at 106.68 106.68 0)
+			(at 101.6 95.25 0)
 			(effects
 				(font
@@
 		)
 		(property "Description" "Mounting Hole without connection"
-			(at 106.68 106.68 0)
+			(at 101.6 95.25 0)
 			(effects
 				(font
@@
 			(project "1026 RPi Power Hat"
 				(path "/0e50632e-8a8b-4b7f-ac56-99c7667bb88a/11547498-585a-4b65-8383-0a98326c007f"
-					(reference "H4")
+					(reference "H2")
 					(unit 1)
 				)
@@
 	)
 	(symbol
+		(lib_id "Mechanical:MountingHole")
+		(at 101.6 107.95 0)
+		(unit 1)
+		(exclude_from_sim no)
+		(in_bom no)
+		(on_board yes)
+		(dnp no)
+		(fields_autoplaced yes)
+		(property "Reference" "H4"
+			(at 104.14 106.7378 0)
+			(effects
+				(font
+					(size 1.27 1.27)
+				)
+				(justify left)
+			)
+		)
+		(property "Value" "MountingHole"
+			(at 104.14 109.1621 0)
+			(effects
+				(font
+					(size 1.27 1.27)
+				)
+				(justify left)
+			)
+		)
+		(property "Footprint" "DW_Mechanical:[MH] MountingHole_2.7mm_M2.5"
+			(at 101.6 107.95 0)
+			(effects
+				(font
+					(size 1.27 1.27)
+				)
+				(hide yes)
+			)
+		)
+		(property "Datasheet" "~"
+			(at 101.6 107.95 0)
+			(effects
+				(font
+					(size 1.27 1.27)
+				)
+				(hide yes)
+			)
+		)
+		(property "Description" "Mounting Hole without connection"
+			(at 101.6 107.95 0)
+			(effects
+				(font
+					(size 1.27 1.27)
+				)
+				(hide yes)
+			)
+		)
+		(instances
+			(project "1026 RPi Power Hat"
+				(path "/0e50632e-8a8b-4b7f-ac56-99c7667bb88a/11547498-585a-4b65-8383-0a98326c007f"
+					(reference "H4")
+					(unit 1)
+				)
+			)
+		)
+	)
+	(symbol
 		(lib_id "DW_Mechanical:Fiducial 1mm-3mm")
 		(at 132.08 107.95 0)
@@
 					(unit 1)
 				)
+			)
+		)
+	)
+	(symbol
+		(lib_id "Mechanical:MountingHole")
+		(at 101.6 101.6 0)
+		(unit 1)
+		(exclude_from_sim no)
+		(in_bom no)
+		(on_board yes)
+		(dnp no)
+		(fields_autoplaced yes)
+		(property "Reference" "H3"
+			(at 104.14 100.3878 0)
+			(effects
+				(font
+					(size 1.27 1.27)
+				)
+				(justify left)
+			)
+		)
+		(property "Value" "MountingHole"
+			(at 104.14 102.8121 0)
+			(effects
+				(font
+					(size 1.27 1.27)
+				)
+				(justify left)
+			)
+		)
+		(property "Footprint" "DW_Mechanical:[MH] MountingHole_2.7mm_M2.5_StencilRegHole"
+			(at 101.6 101.6 0)
+			(effects
+				(font
+					(size 1.27 1.27)
+				)
+				(hide yes)
+			)
+		)
+		(property "Datasheet" "~"
+			(at 101.6 101.6 0)
+			(effects
+				(font
+					(size 1.27 1.27)
+				)
+				(hide yes)
+			)
+		)
+		(property "Description" "Mounting Hole without connection"
+			(at 101.6 101.6 0)
+			(effects
+				(font
+					(size 1.27 1.27)
+				)
+				(hide yes)
+			)
+		)
+		(instances
+			(project "1026 RPi Power Hat"
+				(path "/0e50632e-8a8b-4b7f-ac56-99c7667bb88a/11547498-585a-4b65-8383-0a98326c007f"
+					(reference "H3")
+					(unit 1)
+				)

Commit message: v1.0.0A
Moved all symbols, footprints, and 3D models to local project-specific libraries in /KiCAD Project/Libraries.
Parts:
- FID1, FID2, FID3: footprint Fiducial:Fiducial_1mm_Mask2mm -> 1026-3D:Fiducial_1mm_Mask2mm; symbol DW_Mechanical:Fiducial 1mm-3mm -> 1026-3D:Fiducial 1mm-3mm
- G1, G2: symbol DW_Mechanical:OSHW_Logo -> 1026-3D:OSHW_Logo
- H1, H4: footprint DW_Mechanical:[MH] MountingHole_2.7mm_M2.5 -> 1026-3D:[MH] MountingHole_2.7mm_M2.5; symbol Mechanical:MountingHole -> 1026-3D:MountingHole
- H2, H3: footprint DW_Mechanical:[MH] MountingHole_2.7mm_M2.5_StencilRegHole -> 1026-3D:[MH] MountingHole_2.7mm_M2.5_StencilRegHole; symbol Mechanical:MountingHole -> 1026-3D:MountingHole
- P1: footprint DW_Mechanical:DW_PCB_Logo -> 1026-3D:DW_PCB_Logo; symbol DW_Mechanical:DW_PCB_Logo -> 1026-3D:DW_PCB_Logo
- P2: footprint DW_Mechanical:[G] RPi HAT+ Designator -> 1026-3D:[G] RPi HAT+ Designator; symbol DW_Mechanical:[G] Raspberry Pi HAT+ Designator -> 1026-3D:[G] Raspberry Pi HAT+ Designator
Changed lines of the file:
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@@
 	)
 	(symbol
-		(lib_id "DW_Mechanical:DW_PCB_Logo")
+		(lib_id "1026-3D:DW_PCB_Logo")
 		(at 132.08 91.44 0)
 		(unit 1)
@@
 			)
 		)
-		(property "Footprint" "DW_Mechanical:DW_PCB_Logo"
+		(property "Footprint" "1026-3D:DW_PCB_Logo"
 			(at 132.08 91.44 0)
 			(effects
@@
 	)
 	(symbol
-		(lib_id "Mechanical:MountingHole")
+		(lib_id "1026-3D:MountingHole")
 		(at 101.6 88.9 0)
 		(unit 1)
@@
 			)
 		)
-		(property "Footprint" "DW_Mechanical:[MH] MountingHole_2.7mm_M2.5"
+		(property "Footprint" "1026-3D:[MH] MountingHole_2.7mm_M2.5"
 			(at 101.6 88.9 0)
 			(effects
@@
 	)
 	(symbol
-		(lib_id "DW_Mechanical:Fiducial 1mm-3mm")
+		(lib_id "1026-3D:Fiducial 1mm-3mm")
 		(at 132.08 102.87 0)
 		(unit 1)
@@
 			)
 		)
-		(property "Footprint" "Fiducial:Fiducial_1mm_Mask2mm"
+		(property "Footprint" "1026-3D:Fiducial_1mm_Mask2mm"
 			(at 132.08 102.87 0)
 			(effects
@@
 	)
 	(symbol
-		(lib_id "DW_Mechanical:OSHW_Logo")
+		(lib_id "1026-3D:OSHW_Logo")
 		(at 165.1 101.6 0)
 		(unit 1)
@@
 	)
 	(symbol
-		(lib_id "DW_Mechanical:[G] Raspberry Pi HAT+ Designator")
+		(lib_id "1026-3D:[G] Raspberry Pi HAT+ Designator")
 		(at 132.08 83.82 0)
 		(unit 1)
@@
 			)
 		)
-		(property "Footprint" "DW_Mechanical:[G] RPi HAT+ Designator"
+		(property "Footprint" "1026-3D:[G] RPi HAT+ Designator"
 			(at 132.08 91.44 0)
 			(effects
@@
 	)
 	(symbol
-		(lib_id "Mechanical:MountingHole")
+		(lib_id "1026-3D:MountingHole")
 		(at 101.6 95.25 0)
 		(unit 1)
@@
 			)
 		)
-		(property "Footprint" "DW_Mechanical:[MH] MountingHole_2.7mm_M2.5_StencilRegHole"
+		(property "Footprint" "1026-3D:[MH] MountingHole_2.7mm_M2.5_StencilRegHole"
 			(at 101.6 95.25 0)
 			(effects
@@
 	)
 	(symbol
-		(lib_id "DW_Mechanical:OSHW_Logo")
+		(lib_id "1026-3D:OSHW_Logo")
 		(at 165.1 91.44 0)
 		(unit 1)
@@
 	)
 	(symbol
-		(lib_id "DW_Mechanical:Fiducial 1mm-3mm")
+		(lib_id "1026-3D:Fiducial 1mm-3mm")
 		(at 132.08 97.79 0)
 		(unit 1)
@@
 			)
 		)
-		(property "Footprint" "Fiducial:Fiducial_1mm_Mask2mm"
+		(property "Footprint" "1026-3D:Fiducial_1mm_Mask2mm"
 			(at 132.08 97.79 0)
 			(effects
@@
 	)
 	(symbol
-		(lib_id "Mechanical:MountingHole")
+		(lib_id "1026-3D:MountingHole")
 		(at 101.6 107.95 0)
 		(unit 1)
@@
 			)
 		)
-		(property "Footprint" "DW_Mechanical:[MH] MountingHole_2.7mm_M2.5"
+		(property "Footprint" "1026-3D:[MH] MountingHole_2.7mm_M2.5"
 			(at 101.6 107.95 0)
 			(effects
@@
 	)
 	(symbol
-		(lib_id "DW_Mechanical:Fiducial 1mm-3mm")
+		(lib_id "1026-3D:Fiducial 1mm-3mm")
 		(at 132.08 107.95 0)
 		(unit 1)
@@
 			)
 		)
-		(property "Footprint" "Fiducial:Fiducial_1mm_Mask2mm"
+		(property "Footprint" "1026-3D:Fiducial_1mm_Mask2mm"
 			(at 132.08 107.95 0)
 			(effects
@@
 	)
 	(symbol
-		(lib_id "Mechanical:MountingHole")
+		(lib_id "1026-3D:MountingHole")
 		(at 101.6 101.6 0)
 		(unit 1)
@@
 			)
 		)
-		(property "Footprint" "DW_Mechanical:[MH] MountingHole_2.7mm_M2.5_StencilRegHole"
+		(property "Footprint" "1026-3D:[MH] MountingHole_2.7mm_M2.5_StencilRegHole"
 			(at 101.6 101.6 0)
 			(effects

Commit message: Prep for PCBway
Verified all parts reference local libraries, update font for PCB board title to Noto Sans font, add Noto Sans fonts to project folder, update 3D image for documentation, update documentation for links to both Oshpark and PCBway .zip files.
Parts:
- G1, G2: footprint DW_Mechanical:OSHW_Logo -> 1026-3D:OSHW_Logo
Changed lines of the file:
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@@
 			)
 		)
-		(property "Footprint" "DW_Mechanical:OSHW_Logo"
+		(property "Footprint" "1026-3D:OSHW_Logo"
 			(at 165.1 101.6 0)
 			(effects
@@
 			)
 		)
-		(property "Footprint" "DW_Mechanical:OSHW_Logo"
+		(property "Footprint" "1026-3D:OSHW_Logo"
 			(at 165.1 91.44 0)
 			(effects
